File: MicroHard/_autosave-PowerSupply.kicad_sch (KiCad schematic)
At the start: 0 parts

Commit message: feat: added fpga
Parts:
- added C1, C16, C17, C18, C19, C2: 22u, symbol Device:C
- added C10, C11: 1u, symbol Device:C
- added C12, C14, C15, C6, C7, C8: 100n, symbol Device:C
- added C13, C4, C5: 10u, symbol Device:C
- added C3: 100u, symbol Device:C_Polarized_US
- added C9: 3.3n, symbol Device:C
- added FB1: FerriteBead, symbol Device:FerriteBead
- added JP1, JP2, JP3: Jumper_2_Bridged, symbol Jumper:Jumper_2_Bridged
- added L1, L2: 1.5u, symbol Device:L
- added L3: 2.2u, symbol Device:L
- added R1: 30.1k, symbol Device:R
- added R2, R4, R8: 22.1k, symbol Device:R
- added R3: 6.81k, symbol Device:R
- added R5, R6: 100k, symbol Device:R
- added R7: 73.2k, symbol Device:R
- added R9: 1, symbol Device:R
- added U1: TPS54325, symbol MicroHardLibrary:TPS54325
- added U2: TPS54294, symbol MicroHardLibrary:TPS54294
Connections:
- net POWER_IN: now also C13.2, C14.2, C3.1, C4.1, C5.2, C6.1, C7.2, U1.13 (VIN), U1.14 (VCC), U1.7 (EN), U2.1 (VIN1), U2.16 (VIN2)
- new net: C17.1, C19.1, JP1.1 (A), L2.2, R3.1, U1.1 (VO)
- new net: FB1.2, R9.1
- new net: C12.1, L3.2, U2.14 (SW2)
- new net: C12.2, U2.15 (VBST2)
- new net: C1.1, C2.1, JP2.2 (B), L1.1, R1.1
- new net: C11.1, R6.1, U2.9 (VREG5)
- new net: C16.1, C18.1, JP3.1 (A), L3.1, R7.1
- new net: R1.2, R2.1, U2.7 (VFB1)
- new net: C9.1, U1.4 (SS)
- new net: C10.1, R5.2, U1.3 (VREG5)
- new net: R7.2, R8.1, U2.10 (VFB2)
- new net: C8.2, U2.2 (VBST1)
- new net: C8.1, L1.2, U2.3 (SW1)
- new net: C15.1, L2.1, U1.10 (SW1), U1.11 (SW2)
- new net: C15.2, U1.12 (VBST)
- new net: R3.2, R4.1, U1.2 (VFB)
- new net +1V0: JP1.2 (B)
- new net +1V8: JP2.1 (A)
- new net +3.3V: FB1.1, JP3.2 (B)
- new net +3.3VA: R9.2
- new net EN1.8V: R5.1, U1.6 (PG), U2.5 (EN1)
- new net EN3.3V: R6.2, U2.12 (EN2), U2.6 (PG1)
- new net GND: C1.2, C10.2, C11.2, C13.1, C14.1, C16.2, C17.2, C18.2, C19.2, C2.2, C3.2, C4.2, C5.1, C6.2, C7.1, C9.2, R2.2, R4.2, R8.2, U1.15 (PwPd), U1.5 (GND), U1.8 (PGND1), U1.9 (PGND2), U2.13 (PGND2), U2.17 (PwPd), U2.4 (PGND1), U2.8 (GND)
Other:
- removed sheet MCU
- removed sheet Power Supply
- note added: "1%"
- note added: "Ip>2.8A, Irms>2.1A"
- note added: "Ip>2.9A, Irms>2.1A"
- note added: "Ip>3.5A, Irms>3.1A"
- title: MicroHard Flight Simulator X -> Power Supply
