File: MicroHard/display.kicad_sch (KiCad schematic)
At the start: 4 parts, among them U5 MAX6955AAX+

Commit message: feat: VGA out lines from FPGA drawn
Parts:
- renumbered C57 to C81, C58 to C82, R10 to R27, U5 to U6
Changed lines of the file:
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@@
 		(on_board yes)
 		(dnp no)
-		(property "Reference" "C58"
+		(property "Reference" "C82"
 			(at 207.264 76.2 0)
 			(effects
@@
 			(project ""
 				(path "/578bd531-a491-4b15-a479-460d159ffc14/da2ad706-b813-4c6c-baa2-e38e56e98281"
-					(reference "C58")
+					(reference "C82")
 					(unit 1)
 				)
@@
 		(dnp no)
 		(fields_autoplaced yes)
-		(property "Reference" "U5"
+		(property "Reference" "U6"
 			(at 93.6879 60.96 0)
 			(effects
@@
 			(project ""
 				(path "/578bd531-a491-4b15-a479-460d159ffc14/da2ad706-b813-4c6c-baa2-e38e56e98281"
-					(reference "U5")
+					(reference "U6")
 					(unit 1)
 				)
@@
 		(on_board yes)
 		(dnp no)
-		(property "Reference" "C57"
+		(property "Reference" "C81"
 			(at 195.58 76.454 0)
 			(effects
@@
 			(project ""
 				(path "/578bd531-a491-4b15-a479-460d159ffc14/da2ad706-b813-4c6c-baa2-e38e56e98281"
-					(reference "C57")
+					(reference "C81")
 					(unit 1)
 				)
@@
 		(dnp no)
 		(fields_autoplaced yes)
-		(property "Reference" "R10"
+		(property "Reference" "R27"
 			(at 64.77 73.6599 0)
 			(effects
@@
 			(project ""
 				(path "/578bd531-a491-4b15-a479-460d159ffc14/da2ad706-b813-4c6c-baa2-e38e56e98281"
-					(reference "R10")
+					(reference "R27")
 					(unit 1)
 				)
@@
 		(dnp no)
 		(fields_autoplaced yes)
-		(property "Reference" "#PWR021"
+		(property "Reference" "#PWR044"
 			(at 60.96 90.17 0)
 			(effects
@@
 			(project ""
 				(path "/578bd531-a491-4b15-a479-460d159ffc14/da2ad706-b813-4c6c-baa2-e38e56e98281"
-					(reference "#PWR021")
+					(reference "#PWR044")
 					(unit 1)
 				)
@@
 		(dnp no)
 		(fields_autoplaced yes)
-		(property "Reference" "U5"
+		(property "Reference" "U6"
 			(at 254 76.1999 0)
 			(effects
@@
 			(project ""
 				(path "/578bd531-a491-4b15-a479-460d159ffc14/da2ad706-b813-4c6c-baa2-e38e56e98281"
-					(reference "U5")
+					(reference "U6")
 					(unit 2)
 				)
@@
 		(dnp no)
 		(fields_autoplaced yes)
-		(property "Reference" "#PWR018"
+		(property "Reference" "#PWR045"
 			(at 200.66 88.9 0)
 			(effects
@@
 			(project ""
 				(path "/578bd531-a491-4b15-a479-460d159ffc14/da2ad706-b813-4c6c-baa2-e38e56e98281"
-					(reference "#PWR018")
+					(reference "#PWR045")
 					(unit 1)
 				)

Commit message: feat: finished schematic, TODO: go through checklist
Parts:
- U6: footprint 21-0040_A36+2_MXM -> (none)
Changed lines of the file:
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@@
 			)
 		)
-		(property "Footprint" "21-0040_A36+2_MXM"
+		(property "Footprint" ""
 			(at 72.39 71.12 0)
 			(effects
@@
 			)
 		)
-		(property "Footprint" "21-0040_A36+2_MXM"
+		(property "Footprint" ""
 			(at 219.71 72.39 0)
 			(effects
