File: MicroHard/display.kicad_sch (KiCad schematic)
At the start: 13 parts, among them U6 MAX6955 Display Driver

Commit message: Renumber parts
Parts:
- gave numbers to parts that had none: 9
- renumbered C81 to C72, C82 to C73, R27 to R26, U6 to U5
Changed lines of the file:
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@@
 		(on_board yes)
 		(dnp no)
-		(property "Reference" "C82"
+		(property "Reference" "C73"
 			(at 57.404 99.06 0)
 			(effects
@@
 			(project ""
 				(path "/578bd531-a491-4b15-a479-460d159ffc14/da2ad706-b813-4c6c-baa2-e38e56e98281"
-					(reference "C82")
+					(reference "C73")
 					(unit 1)
 				)
@@
 		(dnp no)
 		(fields_autoplaced yes)
-		(property "Reference" "LED?"
+		(property "Reference" "LED1"
 			(at 50.8 17.78 0)
 			(effects
@@
 			(project ""
 				(path "/578bd531-a491-4b15-a479-460d159ffc14/da2ad706-b813-4c6c-baa2-e38e56e98281"
-					(reference "LED?")
+					(reference "LED1")
 					(unit 1)
 				)
@@
 		(dnp no)
 		(fields_autoplaced yes)
-		(property "Reference" "R?"
+		(property "Reference" "R27"
 			(at 69.85 179.0699 0)
 			(effects
@@
 			(project ""
 				(path "/578bd531-a491-4b15-a479-460d159ffc14/da2ad706-b813-4c6c-baa2-e38e56e98281"
-					(reference "R?")
+					(reference "R27")
 					(unit 1)
 				)
@@
 		(dnp no)
 		(fields_autoplaced yes)
-		(property "Reference" "LED?"
+		(property "Reference" "LED6"
 			(at 250.19 80.01 0)
 			(effects
@@
 			(project "MicroHard"
 				(path "/578bd531-a491-4b15-a479-460d159ffc14/da2ad706-b813-4c6c-baa2-e38e56e98281"
-					(reference "LED?")
+					(reference "LED6")
 					(unit 1)
 				)
@@
 		(dnp no)
 		(fields_autoplaced yes)
-		(property "Reference" "R?"
+		(property "Reference" "R25"
 			(at 53.34 133.3499 0)
 			(effects
@@
 			(project "MicroHard"
 				(path "/578bd531-a491-4b15-a479-460d159ffc14/da2ad706-b813-4c6c-baa2-e38e56e98281"
-					(reference "R?")
+					(reference "R25")
 					(unit 1)
 				)
@@
 		(dnp no)
 		(fields_autoplaced yes)
-		(property "Reference" "LED?"
+		(property "Reference" "LED3"
 			(at 181.61 19.05 0)
 			(effects
@@
 			(project "MicroHard"
 				(path "/578bd531-a491-4b15-a479-460d159ffc14/da2ad706-b813-4c6c-baa2-e38e56e98281"
-					(reference "LED?")
+					(reference "LED3")
 					(unit 1)
 				)
@@
 		(dnp no)
 		(fields_autoplaced yes)
-		(property "Reference" "U6"
+		(property "Reference" "U5"
 			(at 91.1479 121.92 0)
 			(effects
@@
 			(project ""
 				(path "/578bd531-a491-4b15-a479-460d159ffc14/da2ad706-b813-4c6c-baa2-e38e56e98281"
-					(reference "U6")
+					(reference "U5")
 					(unit 1)
 				)
@@
 		(on_board yes)
 		(dnp no)
-		(property "Reference" "C81"
+		(property "Reference" "C72"
 			(at 45.72 99.314 0)
 			(effects
@@
 			(project ""
 				(path "/578bd531-a491-4b15-a479-460d159ffc14/da2ad706-b813-4c6c-baa2-e38e56e98281"
-					(reference "C81")
+					(reference "C72")
 					(unit 1)
 				)
@@
 		(on_board yes)
 		(dnp no)
-		(property "Reference" "C?"
+		(property "Reference" "C74"
 			(at 110.744 177.8 0)
 			(effects
@@
 			(project "MicroHard"
 				(path "/578bd531-a491-4b15-a479-460d159ffc14/da2ad706-b813-4c6c-baa2-e38e56e98281"
-					(reference "C?")
+					(reference "C74")
 					(unit 1)
 				)
@@
 		(dnp no)
 		(fields_autoplaced yes)
-		(property "Reference" "LED?"
+		(property "Reference" "LED2"
 			(at 118.11 17.78 0)
 			(effects
@@
 			(project "MicroHard"
 				(path "/578bd531-a491-4b15-a479-460d159ffc14/da2ad706-b813-4c6c-baa2-e38e56e98281"
-					(reference "LED?")
+					(reference "LED2")
 					(unit 1)
 				)
@@
 		(dnp no)
 		(fields_autoplaced yes)
-		(property "Reference" "R27"
+		(property "Reference" "R26"
 			(at 62.23 133.3499 0)
 			(effects
@@
 			(project ""
 				(path "/578bd531-a491-4b15-a479-460d159ffc14/da2ad706-b813-4c6c-baa2-e38e56e98281"
-					(reference "R27")
+					(reference "R26")
 					(unit 1)
 				)
@@
 		(dnp no)
 		(fields_autoplaced yes)
-		(property "Reference" "LED?"
+		(property "Reference" "LED5"
 			(at 248.92 19.05 0)
 			(effects
@@
 			(project "MicroHard"
 				(path "/578bd531-a491-4b15-a479-460d159ffc14/da2ad706-b813-4c6c-baa2-e38e56e98281"
-					(reference "LED?")
+					(reference "LED5")
 					(unit 1)
 				)
@@
 		(dnp no)
 		(fields_autoplaced yes)
-		(property "Reference" "LED?"
+		(property "Reference" "LED4"
 			(at 181.61 78.74 0)
 			(effects
@@
 			(project "MicroHard"
 				(path "/578bd531-a491-4b15-a479-460d159ffc14/da2ad706-b813-4c6c-baa2-e38e56e98281"
-					(reference "LED?")
+					(reference "LED4")
 					(unit 1)
 				)
@@
 		(dnp no)
 		(fields_autoplaced yes)
-		(property "Reference" "#PWR044"
+		(property "Reference" "#PWR046"
 			(at 58.42 151.13 0)
 			(effects
@@
 			(project ""
 				(path "/578bd531-a491-4b15-a479-460d159ffc14/da2ad706-b813-4c6c-baa2-e38e56e98281"
-					(reference "#PWR044")
+					(reference "#PWR046")
 					(unit 1)
 				)
@@
 		(dnp no)
 		(fields_autoplaced yes)
-		(property "Reference" "U6"
+		(property "Reference" "U5"
 			(at 104.14 99.0599 0)
 			(effects
@@
 			(project ""
 				(path "/578bd531-a491-4b15-a479-460d159ffc14/da2ad706-b813-4c6c-baa2-e38e56e98281"
-					(reference "U6")
+					(reference "U5")
 					(unit 2)
 				)
@@
 		(dnp no)
 		(fields_autoplaced yes)
-		(property "Reference" "#PWR058"
+		(property "Reference" "#PWR048"
 			(at 119.38 189.23 0)
 			(effects
@@
 			(project ""
 				(path "/578bd531-a491-4b15-a479-460d159ffc14/da2ad706-b813-4c6c-baa2-e38e56e98281"
-					(reference "#PWR058")
+					(reference "#PWR048")
 					(unit 1)
 				)
@@
 		(dnp no)
 		(fields_autoplaced yes)
-		(property "Reference" "#PWR057"
+		(property "Reference" "#PWR047"
 			(at 67.31 190.5 0)
 			(effects
@@
 			(project ""
 				(path "/578bd531-a491-4b15-a479-460d159ffc14/da2ad706-b813-4c6c-baa2-e38e56e98281"
-					(reference "#PWR057")
-					(unit 1)
-				)
+					(reference "#PWR047")
+					(unit 1)
+				)

Commit message: Add missing footprint libs
Parts:
- U5: footprint 21-0040_A36+2_MXM -> MAX6955:21-0040_A36&plus_2_MXM
Changed lines of the file:
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@@
 			)
 		)
-		(property "Footprint" "21-0040_A36+2_MXM"
+		(property "Footprint" "MAX6955:21-0040_A36&plus_2_MXM"
 			(at 69.85 132.08 0)
 			(effects
@@
 			)
 		)
-		(property "Footprint" "21-0040_A36+2_MXM"
+		(property "Footprint" "MAX6955:21-0040_A36&plus_2_MXM"
 			(at 69.85 95.25 0)
 			(effects

Commit message: footprints
Parts:
- C72: footprint (none) -> Capacitor_SMD:C_1210_3225Metric_Pad1.33x2.70mm_HandSolder
- C73: footprint (none) -> Capacitor_SMD:C_1206_3216Metric_Pad1.33x1.80mm_HandSolder
- C74: footprint (none) -> Capacitor_SMD:C_0805_2012Metric_Pad1.18x1.45mm_HandSolder
- R25, R26: footprint Resistor_SMD:R_0805_2012Metric_Pad1.20x1.40mm_HandSolder -> Resistor_SMD:R_1206_3216Metric_Pad1.30x1.75mm_HandSolder
- R27: footprint (none) -> Resistor_SMD:R_1206_3216Metric_Pad1.30x1.75mm_HandSolder

Commit message: Initial layout
Parts:
- renumbered LED5 to LED4, LED4 to LED5
Changed lines of the file:
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@@
 		(dnp no)
 		(fields_autoplaced yes)
-		(property "Reference" "LED5"
+		(property "Reference" "LED4"
 			(at 248.92 19.05 0)
 			(effects
@@
 			(project "MicroHard"
 				(path "/578bd531-a491-4b15-a479-460d159ffc14/da2ad706-b813-4c6c-baa2-e38e56e98281"
-					(reference "LED5")
+					(reference "LED4")
 					(unit 1)
 				)
@@
 		(dnp no)
 		(fields_autoplaced yes)
-		(property "Reference" "LED4"
+		(property "Reference" "LED5"
 			(at 181.61 78.74 0)
 			(effects
@@
 			(project "MicroHard"
 				(path "/578bd531-a491-4b15-a479-460d159ffc14/da2ad706-b813-4c6c-baa2-e38e56e98281"
-					(reference "LED4")
+					(reference "LED5")
 					(unit 1)
 				)
@@
 		(dnp no)
 		(fields_autoplaced yes)
-		(property "Reference" "#PWR048"
+		(property "Reference" "#PWR047"
 			(at 119.38 189.23 0)
 			(effects
@@
 			(project ""
 				(path "/578bd531-a491-4b15-a479-460d159ffc14/da2ad706-b813-4c6c-baa2-e38e56e98281"
-					(reference "#PWR048")
+					(reference "#PWR047")
 					(unit 1)
 				)
@@
 		(dnp no)
 		(fields_autoplaced yes)
-		(property "Reference" "#PWR047"
+		(property "Reference" "#PWR048"
 			(at 67.31 190.5 0)
 			(effects
@@
 			(project ""
 				(path "/578bd531-a491-4b15-a479-460d159ffc14/da2ad706-b813-4c6c-baa2-e38e56e98281"
-					(reference "#PWR047")
+					(reference "#PWR048")
 					(unit 1)
 				)

Commit message: VGA and Display layout
Parts:
- added R74: 12k, Resistor_SMD:R_1206_3216Metric_Pad1.30x1.75mm_HandSolder, symbol Device:R
- R27: value 112k -> 100k
Connections:
- net GND: now also R74.2; no longer R27.2
- new net: R27.2, R74.1
Other:
- moved on the sheet: R27
Changed lines of the file:
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@@
 	(wire
 		(pts
-			(xy 67.31 172.72) (xy 67.31 176.53)
+			(xy 67.31 172.72) (xy 67.31 173.99)
 		)
 		(stroke
@@
 	(symbol
 		(lib_id "Device:R")
-		(at 67.31 180.34 0)
+		(at 67.31 177.8 0)
 		(unit 1)
 		(exclude_from_sim no)
@@
 		(fields_autoplaced yes)
 		(property "Reference" "R27"
-			(at 69.85 179.0699 0)
+			(at 69.85 176.5299 0)
 			(effects
 				(font
@@
 			)
 		)
-		(property "Value" "112k"
-			(at 69.85 181.6099 0)
+		(property "Value" "100k"
+			(at 69.85 179.0699 0)
 			(effects
 				(font
@@
 		)
 		(property "Footprint" "Resistor_SMD:R_1206_3216Metric_Pad1.30x1.75mm_HandSolder"
-			(at 65.532 180.34 90)
+			(at 65.532 177.8 90)
 			(effects
 				(font
@@
 		)
 		(property "Datasheet" "~"
-			(at 67.31 180.34 0)
+			(at 67.31 177.8 0)
 			(effects
 				(font
@@
 		)
 		(property "Description" "Resistor"
-			(at 67.31 180.34 0)
+			(at 67.31 177.8 0)
 			(effects
 				(font
@@
 		)
 		(property "Author" ""
-			(at 67.31 180.34 0)
+			(at 67.31 177.8 0)
 			(effects
 				(font
@@
 		)
 		(property "License" ""
-			(at 67.31 180.34 0)
+			(at 67.31 177.8 0)
 			(effects
 				(font
@@
 		)
 		(property "MPN" ""
-			(at 67.31 180.34 0)
+			(at 67.31 177.8 0)
 			(effects
 				(font
@@
 		)
 		(property "Manufacturer" ""
-			(at 67.31 180.34 0)
+			(at 67.31 177.8 0)
 			(effects
 				(font
@@
 		)
 		(property "Tolerance" ""
-			(at 67.31 180.34 0)
+			(at 67.31 177.8 0)
 			(effects
 				(font
@@
 		)
 		(property "Val" ""
-			(at 67.31 180.34 0)
+			(at 67.31 177.8 0)
 			(effects
 				(font
@@
 	)
 	(symbol
+		(lib_id "Device:R")
+		(at 67.31 185.42 0)
+		(unit 1)
+		(exclude_from_sim no)
+		(in_bom yes)
+		(on_board yes)
+		(dnp no)
+		(fields_autoplaced yes)
+		(property "Reference" "R74"
+			(at 69.85 184.1499 0)
+			(effects
+				(font
+					(size 1.27 1.27)
+				)
+				(justify left)
+			)
+		)
+		(property "Value" "12k"
+			(at 69.85 186.6899 0)
+			(effects
+				(font
+					(size 1.27 1.27)
+				)
+				(justify left)
+			)
+		)
+		(property "Footprint" "Resistor_SMD:R_1206_3216Metric_Pad1.30x1.75mm_HandSolder"
+			(at 65.532 185.42 90)
+			(effects
+				(font
+					(size 1.27 1.27)
+				)
+				(hide yes)
+			)
+		)
+		(property "Datasheet" "~"
+			(at 67.31 185.42 0)
+			(effects
+				(font
+					(size 1.27 1.27)
+				)
+				(hide yes)
+			)
+		)
+		(property "Description" "Resistor"
+			(at 67.31 185.42 0)
+			(effects
+				(font
+					(size 1.27 1.27)
+				)
+				(hide yes)
+			)
+		)
+		(property "Author" ""
+			(at 67.31 185.42 0)
+			(effects
+				(font
+					(size 1.27 1.27)
+				)
+				(hide yes)
+			)
+		)
+		(property "License" ""
+			(at 67.31 185.42 0)
+			(effects
+				(font
+					(size 1.27 1.27)
+				)
+				(hide yes)
+			)
+		)
+		(property "MPN" ""
+			(at 67.31 185.42 0)
+			(effects
+				(font
+					(size 1.27 1.27)
+				)
+				(hide yes)
+			)
+		)
+		(property "Manufacturer" ""
+			(at 67.31 185.42 0)
+			(effects
+				(font
+					(size 1.27 1.27)
+				)
+				(hide yes)
+			)
+		)
+		(property "Tolerance" ""
+			(at 67.31 185.42 0)
+			(effects
+				(font
+					(size 1.27 1.27)
+				)
+				(hide yes)
+			)
+		)
+		(property "Val" ""
+			(at 67.31 185.42 0)
+			(effects
+				(font
+					(size 1.27 1.27)
+				)
+				(hide yes)
+			)
+		)
+		(pin "1"
+		)
+		(pin "2"
+		)
+		(instances
+			(project "MicroHard"
+				(path "/578bd531-a491-4b15-a479-460d159ffc14/da2ad706-b813-4c6c-baa2-e38e56e98281"
+					(reference "R74")
+					(unit 1)
+				)
+			)
+		)
+	)
+	(symbol
 		(lib_id "MAX6955:MAX6955AAX+")
 		(at 69.85 95.25 0)
@@
 	(symbol
 		(lib_id "power:GND")
-		(at 67.31 184.15 0)
+		(at 67.31 189.23 0)
 		(unit 1)
 		(exclude_from_sim no)
@@
 		(fields_autoplaced yes)
 		(property "Reference" "#PWR048"
-			(at 67.31 190.5 0)
+			(at 67.31 195.58 0)
 			(effects
 				(font
@@
 		)
 		(property "Value" "GND"
-			(at 67.31 189.23 0)
+			(at 67.31 194.31 0)
 			(effects
 				(font
@@
 		)
 		(property "Footprint" ""
-			(at 67.31 184.15 0)
+			(at 67.31 189.23 0)
 			(effects
 				(font
@@
 		)
 		(property "Datasheet" ""
-			(at 67.31 184.15 0)
+			(at 67.31 189.23 0)
 			(effects
 				(font
@@
 		)
 		(property "Description" "Power symbol creates a global label with name \"GND\" , ground"
-			(at 67.31 184.15 0)
+			(at 67.31 189.23 0)
 			(effects
 				(font

Commit message: Fix wrong display pin connection
Connections:
- net DD_O5: now also LED6.18
- net DD_O6: no longer LED6.18
Changed lines of the file:
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@@
 		)
 	)
-	(global_label "DD_O6"
+	(global_label "DD_O5"
 		(shape input)
 		(at 270.51 107.95 0)

Commit message: Fix schematics for delivery
Parts:
- removed LED1, LED2, LED3, LED4, LED5, LED6: LTP-587HR, LTP-587HR_LTO, symbol LTP-587HR:LTP-587HR
- added LED1, LED2, LED3, LED4, LED5, LED6: PSC05-12GWA, PSC05-12GWA_LTO, symbol PSC05-12GWA:PSC05-12GWA
Connections:
- net DD_O0: now also LED1.18, LED3.2 (A), LED4.2 (A), LED5.2 (A), LED6.2 (A)
- net DD_O1: now also LED2.18, LED3.1 (B), LED4.1 (B), LED5.1 (B), LED6.1 (B)
- net DD_O10: now also LED1.14 (U), LED2.14 (U), LED3.14 (U), LED4.14 (U), LED5.14 (U), LED6.14 (U)
- net DD_O11: now also LED1.15 (P), LED2.15 (P), LED3.15 (P), LED4.15 (P), LED5.15 (P), LED6.15 (P)
- net DD_O12: now also LED1.4 (K), LED2.4 (K), LED3.4 (K), LED4.4 (K), LED5.4 (K), LED6.4 (K)
- net DD_O13: now also LED1.3 (M), LED2.3 (M), LED3.3 (M), LED4.3 (M), LED5.3 (M), LED6.3 (M)
- net DD_O14: now also LED1.17 (N), LED2.17 (N), LED3.17 (N), LED4.17 (N), LED5.17 (N), LED6.17 (N)
- net DD_O15: now also LED1.12 (R), LED2.12 (R), LED3.12 (R), LED4.12 (R), LED5.12 (R), LED6.12 (R)
- net DD_O16: now also LED1.11 (S), LED2.11 (S), LED3.11 (S), LED4.11 (S), LED5.11 (S), LED6.11 (S)
- net DD_O17: now also LED1.7 (T), LED2.7 (T), LED3.7 (T), LED4.7 (T), LED5.7 (T), LED6.7 (T)
- net DD_O18: now also LED1.10 (DP), LED2.10 (DP), LED3.10 (DP), LED4.10 (DP), LED5.10 (DP), LED6.10 (DP)
- net DD_O2: now also LED1.2 (A), LED2.2 (A), LED3.18, LED5.16 (C), LED6.16 (C)
- net DD_O3: now also LED1.1 (B), LED2.1 (B), LED4.18, LED5.13 (D), LED6.13 (D)
- net DD_O4: now also LED1.16 (C), LED2.16 (C), LED3.16 (C), LED4.16 (C), LED5.18
- net DD_O5: now also LED1.13 (D), LED2.13 (D), LED3.13 (D), LED4.13 (D), LED6.18
- net DD_O6: now also LED1.9 (E), LED2.9 (E), LED3.9 (E), LED4.9 (E), LED5.9 (E), LED6.9 (E)
- net DD_O7: now also LED1.8 (F), LED2.8 (F), LED3.8 (F), LED4.8 (F), LED5.8 (F), LED6.8 (F)
- net DD_O8: now also LED1.6 (G), LED2.6 (G), LED3.6 (G), LED4.6 (G), LED5.6 (G), LED6.6 (G)
- net DD_O9: now also LED1.5 (H), LED2.5 (H), LED3.5 (H), LED4.5 (H), LED5.5 (H), LED6.5 (H)
Other:
- company: (none) -> MicroHard
- title: (none) -> Alphanumeric Display
