File: MicroHard/mcu.kicad_sch (KiCad schematic)
At the start: 28 parts, among them J1 GPIO_header, J2 MCU_Debug, J3 Controller Connector, SW1 KMR221NGLFS, SW2 KMR221NGLFS, U3 EFM32GG842F1024, Y1 48MHz

Commit message: Renumber parts
Parts:
- gave numbers to parts that had none: 5
- renumbered D1 to D2, J1 to J2, J2 to J3, J3 to J5, R10 to R11, R11 to R13, R12 to R14, SW1 to SW2, SW2 to SW3
Changed lines of the file:
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@@
 		(dnp no)
 		(fields_autoplaced yes)
-		(property "Reference" "#PWR056"
+		(property "Reference" "#PWR012"
 			(at 29.21 46.99 0)
 			(effects
@@
 			(project "MicroHard"
 				(path "/578bd531-a491-4b15-a479-460d159ffc14/51bb8540-90e7-4b9a-973c-776e3825d084"
-					(reference "#PWR056")
+					(reference "#PWR012")
 					(unit 1)
 				)
@@
 		(on_board yes)
 		(dnp no)
-		(property "Reference" "#PWR016"
+		(property "Reference" "#PWR020"
 			(at 129.54 158.75 0)
 			(effects
@@
 			(project ""
 				(path "/578bd531-a491-4b15-a479-460d159ffc14/51bb8540-90e7-4b9a-973c-776e3825d084"
-					(reference "#PWR016")
+					(reference "#PWR020")
 					(unit 1)
 				)
@@
 		(dnp no)
 		(fields_autoplaced yes)
-		(property "Reference" "R11"
+		(property "Reference" "R13"
 			(at 31.75 67.3099 0)
 			(effects
@@
 			(project ""
 				(path "/578bd531-a491-4b15-a479-460d159ffc14/51bb8540-90e7-4b9a-973c-776e3825d084"
-					(reference "R11")
+					(reference "R13")
 					(unit 1)
 				)
@@
 		(on_board yes)
 		(dnp no)
-		(property "Reference" "R12"
+		(property "Reference" "R14"
 			(at 100.3299 31.75 0)
 			(effects
@@
 			(project ""
 				(path "/578bd531-a491-4b15-a479-460d159ffc14/51bb8540-90e7-4b9a-973c-776e3825d084"
-					(reference "R12")
+					(reference "R14")
 					(unit 1)
 				)
@@
 		(dnp no)
 		(fields_autoplaced yes)
-		(property "Reference" "#PWR013"
+		(property "Reference" "#PWR017"
 			(at 81.28 83.82 0)
 			(effects
@@
 			(project ""
 				(path "/578bd531-a491-4b15-a479-460d159ffc14/51bb8540-90e7-4b9a-973c-776e3825d084"
-					(reference "#PWR013")
+					(reference "#PWR017")
 					(unit 1)
 				)
@@
 		(on_board yes)
 		(dnp no)
-		(property "Reference" "R?"
+		(property "Reference" "R15"
 			(at 108.204 41.656 0)
 			(effects
@@
 			(project "MicroHard"
 				(path "/578bd531-a491-4b15-a479-460d159ffc14/51bb8540-90e7-4b9a-973c-776e3825d084"
-					(reference "R?")
+					(reference "R15")
 					(unit 1)
 				)
@@
 		(dnp no)
 		(fields_autoplaced yes)
-		(property "Reference" "#PWR09"
+		(property "Reference" "#PWR011"
 			(at 27.94 113.03 0)
 			(effects
@@
 			(project ""
 				(path "/578bd531-a491-4b15-a479-460d159ffc14/51bb8540-90e7-4b9a-973c-776e3825d084"
-					(reference "#PWR09")
+					(reference "#PWR011")
 					(unit 1)
 				)
@@
 		(dnp no)
 		(fields_autoplaced yes)
-		(property "Reference" "SW1"
+		(property "Reference" "SW2"
 			(at 43.18 49.53 0)
 			(effects
@@
 			(project ""
 				(path "/578bd531-a491-4b15-a479-460d159ffc14/51bb8540-90e7-4b9a-973c-776e3825d084"
-					(reference "SW1")
+					(reference "SW2")
 					(unit 1)
 				)
@@
 		(dnp no)
 		(fields_autoplaced yes)
-		(property "Reference" "SW?"
+		(property "Reference" "SW1"
 			(at 43.18 17.78 0)
 			(effects
@@
 			(project "MicroHard"
 				(path "/578bd531-a491-4b15-a479-460d159ffc14/51bb8540-90e7-4b9a-973c-776e3825d084"
-					(reference "SW?")
+					(reference "SW1")
 					(unit 1)
 				)
@@
 		(dnp no)
 		(fields_autoplaced yes)
-		(property "Reference" "#PWR020"
+		(property "Reference" "#PWR025"
 			(at 256.54 123.19 0)
 			(effects
@@
 			(project ""
 				(path "/578bd531-a491-4b15-a479-460d159ffc14/51bb8540-90e7-4b9a-973c-776e3825d084"
-					(reference "#PWR020")
+					(reference "#PWR025")
 					(unit 1)
 				)
@@
 		(on_board yes)
 		(dnp no)
-		(property "Reference" "J3"
+		(property "Reference" "J5"
 			(at 263.144 92.71 0)
 			(effects
@@
 			(project ""
 				(path "/578bd531-a491-4b15-a479-460d159ffc14/51bb8540-90e7-4b9a-973c-776e3825d084"
-					(reference "J3")
+					(reference "J5")
 					(unit 1)
 				)
@@
 		(on_board yes)
 		(dnp no)
-		(property "Reference" "J1"
+		(property "Reference" "J2"
 			(at 112.014 90.17 0)
 			(effects
@@
 			(project ""
 				(path "/578bd531-a491-4b15-a479-460d159ffc14/51bb8540-90e7-4b9a-973c-776e3825d084"
-					(reference "J1")
+					(reference "J2")
 					(unit 1)
 				)
@@
 		(dnp no)
 		(fields_autoplaced yes)
-		(property "Reference" "#PWR012"
+		(property "Reference" "#PWR015"
 			(at 64.77 158.75 0)
 			(effects
@@
 			(project ""
 				(path "/578bd531-a491-4b15-a479-460d159ffc14/51bb8540-90e7-4b9a-973c-776e3825d084"
-					(reference "#PWR012")
+					(reference "#PWR015")
 					(unit 1)
 				)
@@
 		(on_board yes)
 		(dnp no)
-		(property "Reference" "D?"
+		(property "Reference" "D3"
 			(at 95.25 40.386 0)
 			(effects
@@
 			(project "MicroHard"
 				(path "/578bd531-a491-4b15-a479-460d159ffc14/51bb8540-90e7-4b9a-973c-776e3825d084"
-					(reference "D?")
+					(reference "D3")
 					(unit 1)
 				)
@@
 		(dnp no)
 		(fields_autoplaced yes)
-		(property "Reference" "R?"
+		(property "Reference" "R12"
 			(at 31.75 35.5599 0)
 			(effects
@@
 			(project "MicroHard"
 				(path "/578bd531-a491-4b15-a479-460d159ffc14/51bb8540-90e7-4b9a-973c-776e3825d084"
-					(reference "R?")
+					(reference "R12")
 					(unit 1)
 				)
@@
 		(dnp no)
 		(fields_autoplaced yes)
-		(property "Reference" "#PWR014"
+		(property "Reference" "#PWR019"
 			(at 88.9 107.95 0)
 			(effects
@@
 			(project ""
 				(path "/578bd531-a491-4b15-a479-460d159ffc14/51bb8540-90e7-4b9a-973c-776e3825d084"
-					(reference "#PWR014")
+					(reference "#PWR019")
 					(unit 1)
 				)
@@
 		(dnp no)
 		(fields_autoplaced yes)
-		(property "Reference" "#PWR018"
+		(property "Reference" "#PWR022"
 			(at 139.7 177.8 0)
 			(effects
@@
 			(project ""
 				(path "/578bd531-a491-4b15-a479-460d159ffc14/51bb8540-90e7-4b9a-973c-776e3825d084"
-					(reference "#PWR018")
+					(reference "#PWR022")
 					(unit 1)
 				)
@@
 		(dnp no)
 		(fields_autoplaced yes)
-		(property "Reference" "#PWR055"
+		(property "Reference" "#PWR018"
 			(at 87.63 44.45 0)
 			(effects
@@
 			(project "MicroHard"
 				(path "/578bd531-a491-4b15-a479-460d159ffc14/51bb8540-90e7-4b9a-973c-776e3825d084"
-					(reference "#PWR055")
+					(reference "#PWR018")
 					(unit 1)
 				)
@@
 		(dnp no)
 		(fields_autoplaced yes)
-		(property "Reference" "SW2"
+		(property "Reference" "SW3"
 			(at 44.45 87.63 0)
 			(effects
@@
 			(project "MicroHard"
 				(path "/578bd531-a491-4b15-a479-460d159ffc14/51bb8540-90e7-4b9a-973c-776e3825d084"
-					(reference "SW2")
+					(reference "SW3")
 					(unit 1)
 				)
@@
 		(dnp no)
 		(fields_autoplaced yes)
-		(property "Reference" "J2"
+		(property "Reference" "J3"
 			(at 209.55 88.9 0)
 			(effects
@@
 			(project ""
 				(path "/578bd531-a491-4b15-a479-460d159ffc14/51bb8540-90e7-4b9a-973c-776e3825d084"
-					(reference "J2")
+					(reference "J3")
 					(unit 1)
 				)
@@
 		(dnp no)
 		(fields_autoplaced yes)
-		(property "Reference" "D1"
+		(property "Reference" "D2"
 			(at 87.3125 27.94 0)
 			(effects
@@
 			(project ""
 				(path "/578bd531-a491-4b15-a479-460d159ffc14/51bb8540-90e7-4b9a-973c-776e3825d084"
-					(reference "D1")
+					(reference "D2")
 					(unit 1)
 				)
@@
 		(dnp no)
 		(fields_autoplaced yes)
-		(property "Reference" "#PWR015"
+		(property "Reference" "#PWR016"
 			(at 81.28 41.91 0)
 			(effects
@@
 			(project ""
 				(path "/578bd531-a491-4b15-a479-460d159ffc14/51bb8540-90e7-4b9a-973c-776e3825d084"
-					(reference "#PWR015")
+					(reference "#PWR016")
 					(unit 1)
 				)
@@
 		(dnp no)
 		(fields_autoplaced yes)
-		(property "Reference" "#PWR019"
+		(property "Reference" "#PWR024"
 			(at 219.71 125.73 0)
 			(effects
@@
 			(project ""
 				(path "/578bd531-a491-4b15-a479-460d159ffc14/51bb8540-90e7-4b9a-973c-776e3825d084"
-					(reference "#PWR019")
+					(reference "#PWR024")
 					(unit 1)
 				)
@@
 		(dnp no)
 		(fields_autoplaced yes)
-		(property "Reference" "#PWR011"
+		(property "Reference" "#PWR014"
 			(at 58.42 195.58 0)
 			(effects
@@
 			(project ""
 				(path "/578bd531-a491-4b15-a479-460d159ffc14/51bb8540-90e7-4b9a-973c-776e3825d084"
-					(reference "#PWR011")
+					(reference "#PWR014")
 					(unit 1)
 				)
@@
 		(dnp no)
 		(fields_autoplaced yes)
-		(property "Reference" "#PWR060"
+		(property "Reference" "#PWR023"
 			(at 214.63 69.85 0)
 			(effects
@@
 			(project ""
 				(path "/578bd531-a491-4b15-a479-460d159ffc14/51bb8540-90e7-4b9a-973c-776e3825d084"
-					(reference "#PWR060")
+					(reference "#PWR023")
 					(unit 1)
 				)
@@
 		(dnp no)
 		(fields_autoplaced yes)
-		(property "Reference" "#PWR059"
+		(property "Reference" "#PWR026"
 			(at 264.16 68.58 0)
 			(effects
@@
 			(project ""
 				(path "/578bd531-a491-4b15-a479-460d159ffc14/51bb8540-90e7-4b9a-973c-776e3825d084"
-					(reference "#PWR059")
+					(reference "#PWR026")
 					(unit 1)
 				)
@@
 		(dnp no)
 		(fields_autoplaced yes)
-		(property "Reference" "R10"
+		(property "Reference" "R11"
 			(at 30.48 87.6299 0)
 			(effects
@@
 			(project "MicroHard"
 				(path "/578bd531-a491-4b15-a479-460d159ffc14/51bb8540-90e7-4b9a-973c-776e3825d084"
-					(reference "R10")
+					(reference "R11")
 					(unit 1)
 				)
@@
 		(dnp no)
 		(fields_autoplaced yes)
-		(property "Reference" "#PWR010"
+		(property "Reference" "#PWR013"
 			(at 29.21 78.74 0)
 			(effects
@@
 			(project ""
 				(path "/578bd531-a491-4b15-a479-460d159ffc14/51bb8540-90e7-4b9a-973c-776e3825d084"
-					(reference "#PWR010")
+					(reference "#PWR013")
 					(unit 1)
 				)
@@
 		(dnp no)
 		(fields_autoplaced yes)
-		(property "Reference" "#PWR017"
+		(property "Reference" "#PWR021"
 			(at 129.54 187.96 0)
 			(effects
@@
 			(project ""
 				(path "/578bd531-a491-4b15-a479-460d159ffc14/51bb8540-90e7-4b9a-973c-776e3825d084"
-					(reference "#PWR017")
+					(reference "#PWR021")
 					(unit 1)
 				)
@@
 		(dnp no)
 		(fields_autoplaced yes)
-		(property "Reference" "J?"
+		(property "Reference" "J4"
 			(at 243.205 26.67 0)
 			(effects
@@
 			(project ""
 				(path "/578bd531-a491-4b15-a479-460d159ffc14/51bb8540-90e7-4b9a-973c-776e3825d084"
-					(reference "J?")
-					(unit 1)
-				)
+					(reference "J4")
+					(unit 1)
+				)

Commit message: footprints
Parts:
- C20, C22, C23, C25, C29, C30: footprint (none) -> Capacitor_SMD:C_1206_3216Metric_Pad1.33x1.80mm_HandSolder
- C21, C24, C26, C31: value 0.1u -> 100n; footprint (none) -> Capacitor_SMD:C_1206_3216Metric_Pad1.33x1.80mm_HandSolder
- J5: footprint (none) -> Connector_PinHeader_2.54mm:PinHeader_1x07_P2.54mm_Vertical
- R11, R12, R13: footprint Resistor_SMD:R_0805_2012Metric_Pad1.20x1.40mm_HandSolder -> Resistor_SMD:R_1206_3216Metric_Pad1.30x1.75mm_HandSolder
- SW1, SW2, SW3: footprint KMR221_CNK -> KMR221NG:KMR221_CNK
