File: MicroHard/MicroHard.kicad_pcb (KiCad board)
At the start: 6 copper layers, 222 x 144.5 mm, 191 parts, among them IC1 IS66WVO32M8DBLL-166BLI, J1 USB_B_Micro, J2 Micro_SD_Card_Det2, J3 GPIO_header, J4 MCU_Debug, J5 Controller Connector, J6 FPGA_GPIO_header, J7 FPGA_DEBUG, J8 L77HDE15SD1CH4FVGA, SW1 KMR221NGLFS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

Commit message: finished FPGA
Parts:
- added C58: 470n, Capacitor_SMD:C_0603_1608Metric_Pad1.08x0.95mm_HandSolder, B.Cu at (112.1, 101.0)
- moved J6 12.4 mm to (171.8, 76.6)
Connections:
- U4 pad D11: Net-(J6-Pin_3) -> unconnected-(U4A-IO_L14N_T2_SRCC_15-PadD11)
- U4 pad D14: Net-(J6-Pin_4) -> unconnected-(U4A-IO_L15P_T2_DQS_15-PadD14)
- U4 pad D15: Net-(J6-Pin_5) -> unconnected-(U4A-IO_L15N_T2_DQS_ADV_B_15-PadD15)
- U4 pad E11: Net-(J6-Pin_2) -> unconnected-(U4A-IO_L14P_T2_SRCC_15-PadE11)
- U4 pad E12: Net-(J6-Pin_1) -> unconnected-(U4A-IO_L13P_T2_MRCC_15-PadE12)
- U4 pad E16: Net-(J6-Pin_8) -> unconnected-(U4A-IO_L17P_T2_A26_15-PadE16)
- U4 pad F12: Net-(J6-Pin_6) -> unconnected-(U4A-IO_L16P_T2_A28_15-PadF12)
- U4 pad F13: Net-(J6-Pin_7) -> unconnected-(U4A-IO_L16N_T2_A27_15-PadF13)
- U4 pad M16: unconnected-(U4A-IO_L7P_T1_D09_14-PadM16) -> FPGA_GPIO0
- U4 pad N14: unconnected-(U4A-IO_L12P_T1_MRCC_14-PadN14) -> Net-(J6-Pin_2)
- U4 pad N16: unconnected-(U4A-IO_L7N_T1_D10_14-PadN16) -> FPGA_GPIO1
- U4 pad P13: unconnected-(U4A-IO_L11N_T1_SRCC_14-PadP13) -> Net-(J6-Pin_3)
- U4 pad P14: unconnected-(U4A-IO_L12N_T1_MRCC_14-PadP14) -> Net-(J6-Pin_1)
- U4 pad P16: unconnected-(U4A-IO_L8N_T1_D12_14-PadP16) -> Net-(J6-Pin_4)
- U4 pad R15: unconnected-(U4A-IO_L9P_T1_DQS_14-PadR15) -> Net-(J6-Pin_8)
- U4 pad R16: unconnected-(U4A-IO_L9N_T1_DQS_D13_14-PadR16) -> Net-(J6-Pin_7)
- U4 pad T14: unconnected-(U4A-IO_L10P_T1_D14_14-PadT14) -> Net-(J6-Pin_6)
- U4 pad T15: unconnected-(U4A-IO_L10N_T1_D15_14-PadT15) -> Net-(J6-Pin_5)
Routing:
- net +3.3VA: track 0.00 -> 119.2 mm, vias 0 -> 1
- net +1V8: track 11.6 -> 123.2 mm
- net FPGA_RESET: track 85.0 -> 191.5 mm, vias 4 -> 3
- net FPGA_DONE: track 68.4 -> 148.8 mm, vias 5 -> 4
- net FPGA_US0_TX: track 24.2 -> 104.5 mm, vias 0 -> 2
- net FPGA_GPIO1: track 12.2 -> 92.3 mm, vias 0 -> 2
- net FPGA_GPIO0: track 12.0 -> 91.3 mm, vias 0 -> 2
- net FPGA_US0_CLK: track 21.4 -> 97.6 mm, vias 0 -> 2
- net FPGA_US0_CS: track 20.5 -> 94.6 mm, vias 0 -> 2
- net Net-(J6-Pin_1): track 0.00 -> 70.9 mm, vias 0 -> 1
- net FPGA_US0_RX: track 22.6 -> 92.6 mm, vias 0 -> 2
- net Net-(J6-Pin_3): track 0.00 -> 69.6 mm, vias 0 -> 1
- net Net-(J6-Pin_2): track 0.00 -> 61.9 mm, vias 0 -> 2
- net Net-(J6-Pin_6): track 0.00 -> 58.6 mm
- net Net-(J6-Pin_5): track 0.00 -> 58.1 mm
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
Commit message: finished layout
Parts:
- moved R15 31.9 mm to (220.8, 77.2)
- moved SW3 31.9 mm to (220.8, 85.2)
- moved TP1 30.6 mm to (140.6, 118.0)
- moved R16 27.4 mm to (142.0, 118.6), turned to -90 degrees
- moved TP2 25.5 mm to (132.4, 135.9)
- moved U1 25.4 mm to (57.2, 99.8)
- moved JP1 25.4 mm to (79.5, 107.3)
- moved R7 25.4 mm to (62.8, 123.9)
- moved C1 25.4 mm to (61.6, 99.6)
- moved C10 25.4 mm to (53.5, 131.9)
- moved C11 25.4 mm to (50.2, 131.9)
- moved C12 25.4 mm to (53.8, 115.9)
- moved C13 25.4 mm to (54.4, 127.4)
- moved C14 25.4 mm to (54.5, 120.4)
- moved C15 25.4 mm to (70.8, 131.9)
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Routing:
- net +3.3VA: track 119.2 -> 7.64 mm
- net I2C0_SDA: track 32.8 -> 136.0 mm, vias 1 -> 2
- net I2C0_SCL: track 29.5 -> 130.2 mm, vias 1 -> 2
- net FPGA_RESET: track 191.5 -> 141.6 mm
- net +1V8: track 123.2 -> 76.8 mm
- net FPGA_DONE: track 148.8 -> 119.2 mm
- net +1V0: track 71.2 -> 48.8 mm
- net SD_US2_RX: track 20.4 -> 39.4 mm, vias 1 -> 2
- net Net-(J3-Pin_5): track 6.76 -> 25.1 mm
- net MCU_Reset: track 41.9 -> 60.0 mm, vias 1 -> 2
- net Net-(J3-Pin_8): track 10.4 -> 26.2 mm
- net SD_US2_CLK: track 21.6 -> 37.2 mm, vias 1 -> 2
- net Net-(J3-Pin_6): track 9.01 -> 24.5 mm
- net Net-(J3-Pin_7): track 10.3 -> 25.3 mm
- net INIT: track 43.5 -> 29.1 mm
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
Commit message: Clean up
Parts:
- added G***: LOGO, LOGO, F.Cu at (187.5, 84.5)
- R18, R19, R75: moved to F.Cu
- moved J6 23.7 mm to (160.0, 100.1), turned to 180 degrees
- moved R15 8.79 mm to (229.5, 78.5), turned to 90 degrees
- moved SW3 7.70 mm to (224.5, 78.5)
- moved J5 6.90 mm to (187.9, 140.5)
- moved R75 6.27 mm to (111.0, 132.0), turned to 0 degrees
- moved J2 5.12 mm to (223.7, 132.8)
- moved R77 5.12 mm to (212.2, 140.2)
- moved C82 5.12 mm to (218.9, 130.9)
- moved R78 5.12 mm to (212.2, 127.7)
- moved R19 4.94 mm to (111.0, 124.1), turned to 0 degrees
- moved J3 4.10 mm to (229.1, 116.5)
- moved J4 4.10 mm to (228.8, 85.7)
- moved R18 3.67 mm to (111.0, 128.0), turned to 0 degrees
- moved J7 2.20 mm to (101.1, 129.0)
- moved C47 1.39 mm to (111.5, 116.6)
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Connections:
- U2 pad V: (no net) -> GND
Routing:
- net +3.3VA: track 7.64 -> 119.0 mm, vias 1 -> 0
- net Net-(J6-Pin_1): track 67.4 -> 40.4 mm, vias 1 -> 2
- net Net-(J6-Pin_3): track 64.0 -> 47.3 mm, vias 1 -> 2
- net Net-(J6-Pin_2): track 55.9 -> 43.4 mm
- net MCU_Reset: track 60.0 -> 71.1 mm
- net +3.3V: track 186.7 -> 177.0 mm, vias 50 -> 52
- net Net-(J6-Pin_6): track 53.5 -> 63.0 mm, vias 0 -> 1
- net GND: track 256.8 -> 265.9 mm, vias 139 -> 141
- net Net-(J6-Pin_4): track 53.7 -> 45.1 mm, vias 0 -> 1
- net Controller_Z: track 26.1 -> 33.1 mm
- net Controller_X: track 27.1 -> 34.1 mm
- net Controller_Btn2: track 20.9 -> 27.7 mm
- net Controller_Btn1: track 20.0 -> 26.8 mm
- net /FPGA/FPGA Config/JTAG_TDI: track 41.9 -> 35.9 mm
- net SD_US2_CLK: track 37.2 -> 42.5 mm
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Other:
- board size 222 x 144.5 mm -> 198.2 x 104.1 mm
- board text added: "Andreas Virkesdal Jonsterhaug Arash Farzaneh Taleghani Bård Raddum Wikmark Eivind Nesje Ian McGregor Aksum Morten Sørensen Viljan van Raaij"
- board text removed: "FPGA Reset"

Commit message: Fix vias
Parts:
- C80: moved to F.Cu
- moved C35 30.8 mm to (99.3, 114.6)
- moved C44 25.1 mm to (101.3, 116.6)
- moved TP2 15.3 mm to (117.6, 132.1)
- moved C43 12.7 mm to (117.4, 95.0), turned to 180 degrees
- moved C39 10.3 mm to (124.2, 98.1)
- moved R71 9.25 mm to (143.3, 100.1), turned to 0 degrees
- moved R70 9.20 mm to (137.8, 100.1), turned to 180 degrees
- moved C1 8.35 mm to (61.0, 107.9)
- moved C12 8.35 mm to (53.1, 124.2)
- moved C17 8.35 mm to (70.0, 124.2)
- moved C18 8.35 mm to (66.2, 124.2)
- moved C19 8.35 mm to (60.9, 132.3)
- moved C2 8.35 mm to (44.6, 108.2)
- moved C3 8.35 mm to (51.4, 116.2)
- moved C4 8.35 mm to (54.6, 116.2)
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Routing:
- net FPGA_LED0: track 70.8 -> 37.2 mm
- net FPGA_LED1: track 70.5 -> 40.6 mm
- net VGA_B3: track 114.5 -> 87.6 mm, vias 3 -> 2
- net FPGA_LED2: track 70.2 -> 47.8 mm
- net VGA_B2: track 112.9 -> 92.7 mm, vias 3 -> 2
- net FPGA_RESET: track 141.4 -> 123.3 mm, vias 3 -> 4
- net VGA_B1: track 108.6 -> 94.4 mm
- net Net-(J6-Pin_6): track 63.0 -> 50.7 mm
- net GND: track 265.9 -> 253.8 mm, vias 141 -> 138
- net INIT: track 29.1 -> 17.3 mm
- net VGA_B0: track 109.7 -> 100.0 mm, vias 3 -> 2
- net VGA_R2: track 82.5 -> 74.0 mm
- net FPGA_US0_CLK: track 85.6 -> 77.2 mm
- net SRAM_DQ2: track 28.7 -> 20.5 mm
- net +3.3VA: track 119.0 -> 111.0 mm
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