File: MicroHard/FPGA.kicad_sch (KiCad schematic)
At the start: 1 part, among them SW4 KMR221NGLFS

Commit message: footprints
Parts:
- SW4: footprint (none) -> KMR221NG:KMR221_CNK
Changed lines of the file:
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@@
 			)
 		)
-		(property "Footprint" ""
+		(property "Footprint" "KMR221NG:KMR221_CNK"
 			(at 35.56 114.3 0)
 			(effects
@@
 			(at 35.56 114.3 0)
 			(effects
+				(font
+					(size 1.27 1.27)
+				)
+				(hide yes)
+			)
+		)
+		(property "Author" ""
+			(at 35.56 114.3 0)
+			(effects
+				(font
+					(size 1.27 1.27)
+				)
+				(hide yes)
+			)
+		)
+		(property "License" ""
+			(at 35.56 114.3 0)
+			(effects
+				(font
+					(size 1.27 1.27)
+				)
+				(hide yes)
+			)
+		)
+		(property "MPN" ""
+			(at 35.56 114.3 0)
+			(effects
+				(font
+					(size 1.27 1.27)
+				)
+				(hide yes)
+			)
+		)
+		(property "Manufacturer" ""
+			(at 35.56 114.3 0)
+			(effects
+				(font
+					(size 1.27 1.27)
+				)
+				(hide yes)
+			)
+		)
+		(property "Tolerance" ""
+			(at 35.56 114.3 0)
+			(effects
+				(font
+					(size 1.27 1.27)
+				)
+				(hide yes)
+			)
+		)
+		(property "Val" ""
+			(at 35.56 114.3 0)
+			(effects

Commit message: Fix schematics for delivery
Other:
- company: (none) -> MicroHard
- title: (none) -> FPGA
