File: MicroHard/FPGA1.kicad_sch (KiCad schematic)
At the start: 18 parts, among them J6 FPGA_GPIO_header, U4 XC7A100T-FTG256, Y2 CB3-3C-20M000000

Commit message: footprints
Parts:
- C32, C46: footprint (none) -> Capacitor_SMD:C_1210_3225Metric_Pad1.33x2.70mm_HandSolder
- C33, C35, C44, C45: footprint (none) -> Capacitor_SMD:C_0805_2012Metric_Pad1.18x1.45mm_HandSolder
- C34: footprint (none) -> Capacitor_SMD:C_1206_3216Metric_Pad1.33x1.80mm_HandSolder
- C36, C37, C38, C39, C40, C41, C42, C43: footprint (none) -> Capacitor_SMD:C_0603_1608Metric_Pad1.08x0.95mm_HandSolder

Commit message: Initial layout
Parts:
- renumbered C35 to C34, C36 to C35, C37 to C36, C38 to C37, C39 to C38, C40 to C39, C42 to C40, C44 to C41, C46 to C42, C41 to C43, C43 to C44, C34 to C46
Changed lines of the file:
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@@
 		(on_board yes)
 		(dnp no)
-		(property "Reference" "C42"
+		(property "Reference" "C40"
 			(at 248.92 18.542 0)
 			(effects
@@
 			(project "MicroHard"
 				(path "/578bd531-a491-4b15-a479-460d159ffc14/e381883e-e672-4900-88a5-08b94f970a88/1131f32d-45e2-48d4-a5b0-b9e8f8db47f2"
-					(reference "C42")
+					(reference "C40")
 					(unit 1)
 				)
@@
 		(on_board yes)
 		(dnp no)
-		(property "Reference" "C39"
+		(property "Reference" "C38"
 			(at 125.984 19.05 0)
 			(effects
@@
 			(project "MicroHard"
 				(path "/578bd531-a491-4b15-a479-460d159ffc14/e381883e-e672-4900-88a5-08b94f970a88/1131f32d-45e2-48d4-a5b0-b9e8f8db47f2"
-					(reference "C39")
+					(reference "C38")
 					(unit 1)
 				)
@@
 		(on_board yes)
 		(dnp no)
-		(property "Reference" "C43"
+		(property "Reference" "C44"
 			(at 254.254 26.162 0)
 			(effects
@@
 			(project "MicroHard"
 				(path "/578bd531-a491-4b15-a479-460d159ffc14/e381883e-e672-4900-88a5-08b94f970a88/1131f32d-45e2-48d4-a5b0-b9e8f8db47f2"
-					(reference "C43")
+					(reference "C44")
 					(unit 1)
 				)
@@
 		(dnp no)
 		(fields_autoplaced yes)
-		(property "Reference" "#PWR029"
+		(property "Reference" "#PWR031"
 			(at 49.53 83.82 0)
 			(effects
@@
 			(project "MicroHard"
 				(path "/578bd531-a491-4b15-a479-460d159ffc14/e381883e-e672-4900-88a5-08b94f970a88/1131f32d-45e2-48d4-a5b0-b9e8f8db47f2"
-					(reference "#PWR029")
+					(reference "#PWR031")
 					(unit 1)
 				)
@@
 		(on_board yes)
 		(dnp no)
-		(property "Reference" "C46"
+		(property "Reference" "C42"
 			(at 271.272 17.78 0)
 			(effects
@@
 			(project "MicroHard"
 				(path "/578bd531-a491-4b15-a479-460d159ffc14/e381883e-e672-4900-88a5-08b94f970a88/1131f32d-45e2-48d4-a5b0-b9e8f8db47f2"
-					(reference "C46")
+					(reference "C42")
 					(unit 1)
 				)
@@
 		(on_board yes)
 		(dnp no)
-		(property "Reference" "C34"
+		(property "Reference" "C46"
 			(at 60.452 85.09 90)
 			(effects
@@
 			(project "MicroHard"
 				(path "/578bd531-a491-4b15-a479-460d159ffc14/e381883e-e672-4900-88a5-08b94f970a88/1131f32d-45e2-48d4-a5b0-b9e8f8db47f2"
-					(reference "C34")
+					(reference "C46")
 					(unit 1)
 				)
@@
 		(on_board yes)
 		(dnp no)
-		(property "Reference" "C44"
+		(property "Reference" "C41"
 			(at 264.414 18.288 0)
 			(effects
@@
 			(project "MicroHard"
 				(path "/578bd531-a491-4b15-a479-460d159ffc14/e381883e-e672-4900-88a5-08b94f970a88/1131f32d-45e2-48d4-a5b0-b9e8f8db47f2"
-					(reference "C44")
+					(reference "C41")
 					(unit 1)
 				)
@@
 		(dnp no)
 		(fields_autoplaced yes)
-		(property "Reference" "#PWR031"
+		(property "Reference" "#PWR030"
 			(at 128.27 58.42 0)
 			(effects
@@
 			(project ""
 				(path "/578bd531-a491-4b15-a479-460d159ffc14/e381883e-e672-4900-88a5-08b94f970a88/1131f32d-45e2-48d4-a5b0-b9e8f8db47f2"
-					(reference "#PWR031")
+					(reference "#PWR030")
 					(unit 1)
 				)
@@
 		(on_board yes)
 		(dnp no)
-		(property "Reference" "C41"
+		(property "Reference" "C43"
 			(at 241.3 26.67 0)
 			(effects
@@
 			(project "MicroHard"
 				(path "/578bd531-a491-4b15-a479-460d159ffc14/e381883e-e672-4900-88a5-08b94f970a88/1131f32d-45e2-48d4-a5b0-b9e8f8db47f2"
-					(reference "C41")
+					(reference "C43")
 					(unit 1)
 				)
@@
 		(on_board yes)
 		(dnp no)
-		(property "Reference" "C36"
+		(property "Reference" "C35"
 			(at 88.9 19.05 0)
 			(effects
@@
 			(project "MicroHard"
 				(path "/578bd531-a491-4b15-a479-460d159ffc14/e381883e-e672-4900-88a5-08b94f970a88/1131f32d-45e2-48d4-a5b0-b9e8f8db47f2"
-					(reference "C36")
+					(reference "C35")
 					(unit 1)
 				)
@@
 		(dnp no)
 		(fields_autoplaced yes)
-		(property "Reference" "#PWR032"
+		(property "Reference" "#PWR029"
 			(at 271.78 43.18 0)
 			(effects
@@
 			(project "MicroHard"
 				(path "/578bd531-a491-4b15-a479-460d159ffc14/e381883e-e672-4900-88a5-08b94f970a88/1131f32d-45e2-48d4-a5b0-b9e8f8db47f2"
-					(reference "#PWR032")
+					(reference "#PWR029")
 					(unit 1)
 				)
@@
 		(on_board yes)
 		(dnp no)
-		(property "Reference" "C35"
+		(property "Reference" "C34"
 			(at 75.184 19.05 0)
 			(effects
@@
 			(project "MicroHard"
 				(path "/578bd531-a491-4b15-a479-460d159ffc14/e381883e-e672-4900-88a5-08b94f970a88/1131f32d-45e2-48d4-a5b0-b9e8f8db47f2"
-					(reference "C35")
+					(reference "C34")
 					(unit 1)
 				)
@@
 		(dnp no)
 		(fields_autoplaced yes)
-		(property "Reference" "#PWR030"
+		(property "Reference" "#PWR032"
 			(at 78.74 110.49 0)
 			(effects
@@
 			(project ""
 				(path "/578bd531-a491-4b15-a479-460d159ffc14/e381883e-e672-4900-88a5-08b94f970a88/1131f32d-45e2-48d4-a5b0-b9e8f8db47f2"
-					(reference "#PWR030")
+					(reference "#PWR032")
 					(unit 1)
 				)
@@
 		(on_board yes)
 		(dnp no)
-		(property "Reference" "C37"
+		(property "Reference" "C36"
 			(at 100.33 19.05 0)
 			(effects
@@
 			(project "MicroHard"
 				(path "/578bd531-a491-4b15-a479-460d159ffc14/e381883e-e672-4900-88a5-08b94f970a88/1131f32d-45e2-48d4-a5b0-b9e8f8db47f2"
-					(reference "C37")
+					(reference "C36")
 					(unit 1)
 				)
@@
 		(on_board yes)
 		(dnp no)
-		(property "Reference" "C40"
+		(property "Reference" "C39"
 			(at 233.934 19.05 0)
 			(effects
@@
 			(project "MicroHard"
 				(path "/578bd531-a491-4b15-a479-460d159ffc14/e381883e-e672-4900-88a5-08b94f970a88/1131f32d-45e2-48d4-a5b0-b9e8f8db47f2"
-					(reference "C40")
+					(reference "C39")
 					(unit 1)
 				)
@@
 		(on_board yes)
 		(dnp no)
-		(property "Reference" "C38"
+		(property "Reference" "C37"
 			(at 113.03 19.05 0)
 			(effects
@@
 			(project "MicroHard"
 				(path "/578bd531-a491-4b15-a479-460d159ffc14/e381883e-e672-4900-88a5-08b94f970a88/1131f32d-45e2-48d4-a5b0-b9e8f8db47f2"
-					(reference "C38")
+					(reference "C37")
 					(unit 1)
 				)

Commit message: VGA and Display layout
Parts:
- J6: footprint Connector_JST:JST_XH_B8B-XH-AM_1x08_P2.50mm_Vertical -> Connector_PinHeader_2.54mm:PinHeader_1x08_P2.54mm_Vertical
Changed lines of the file:
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@@
 			)
 		)
-		(property "Footprint" "Connector_JST:JST_XH_B8B-XH-AM_1x08_P2.50mm_Vertical"
+		(property "Footprint" "Connector_PinHeader_2.54mm:PinHeader_1x08_P2.54mm_Vertical"
 			(at 280.67 110.49 0)
 			(effects

Commit message: finished FPGA
Connections:
- net at U4.D11 (IO_L14N_T2_SRCC_15): no longer J6.3 (Pin_3)
- net at U4.D14 (IO_L15P_T2_DQS_15): no longer J6.4 (Pin_4)
- net at U4.D15 (IO_L15N_T2_DQS_ADV_B_15): no longer J6.5 (Pin_5)
- net at U4.E11 (IO_L14P_T2_SRCC_15): no longer J6.2 (Pin_2)
- net at U4.E12 (IO_L13P_T2_MRCC_15): no longer J6.1 (Pin_1)
- net at U4.E16 (IO_L17P_T2_A26_15): no longer J6.8 (Pin_8)
- net at U4.F12 (IO_L16P_T2_A28_15): no longer J6.6 (Pin_6)
- net at U4.F13 (IO_L16N_T2_A27_15): no longer J6.7 (Pin_7)
- net FPGA_GPIO0: now reaches U4.M16 (IO_L7P_T1_D09_14)
- net at U4.N14 (IO_L12P_T1_MRCC_14): now also J6.2 (Pin_2)
- net FPGA_GPIO1: now reaches U4.N16 (IO_L7N_T1_D10_14)
- net at U4.P13 (IO_L11N_T1_SRCC_14): now also J6.3 (Pin_3)
- net at U4.P14 (IO_L12N_T1_MRCC_14): now also J6.1 (Pin_1)
- net at U4.P16 (IO_L8N_T1_D12_14): now also J6.4 (Pin_4)
- net at U4.R15 (IO_L9P_T1_DQS_14): now also J6.8 (Pin_8)
- net at U4.R16 (IO_L9N_T1_DQS_D13_14): now also J6.7 (Pin_7)
- net at U4.T14 (IO_L10P_T1_D14_14): now also J6.6 (Pin_6)
- net at U4.T15 (IO_L10N_T1_D15_14): now also J6.5 (Pin_5)
- no-connect marks 50 -> 48

Commit message: Fix schematics for delivery
Other:
- company: (none) -> MicroHard
- title: (none) -> FPGA Unit A
