File: MicroHard/FPGA4.kicad_sch (KiCad schematic)
At the start: 25 parts, among them U4 XC7A100T-FTG256

Commit message: Initial layout
Parts:
- renumbered C52 to C49, C55 to C50, C58 to C51, C60 to C52, C62 to C53, C63 to C54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

Commit message: Fix schematics for delivery
Other:
- company: (none) -> MicroHard
- title: (none) -> FPGA Power Supply
