File: MicroHard/vga_out_sch.kicad_sch (KiCad schematic)
At the start: 21 parts, among them U7 SN74ALVC245PWR, U8 SN74ALVC245PWR

Commit message: feat: finished schematic, TODO: go through checklist
Parts:
- removed J?: 1-1734530-3, CONN_1-1734530-1_TYCO, symbol VGA PORT:1-1734530-3
- added J5: 1-1734530-3, MicroHard:CONN_1-1734530-1_TYCO, symbol VGA PORT:1-1734530-3
- added R35, R36, R37, R38, R42, R43, R44, R45, R46, R50, R51, R52, R53, R54, R58: 536, symbol Device:R
- added R39, R40, R41, R47, R48, R49, R55, R56, R57: 270, symbol Device:R
- added R59, R60: 100, symbol Device:R
- U7, U8: footprint PW20 -> footprints:PW20
- gave numbers to parts that had none: 18
Connections:
- net +3.3V: now also U8.1 (DIR)
- net B0: now also R54.1
- net B1: now also R53.1
- net B2: now also R52.1
- net B3: now also R51.1
- net G0: now also R46.1
- net G1: now also R45.1
- net G2: now also R44.1
- net G3: now also R43.1
- net GND: now also J5.10, J5.5, J5.6, J5.7, J5.8, R42.2, R50.2, R58.2
- net HSYNC: now also R59.2
- net R0: now also R38.1
- net R1: now also R37.1
- net R2: now also R36.1
- net R3: now also R35.1
- net VSYNC: now also R60.2
- new net: R46.2, R49.2, R50.1
- new net: J5.1, R35.2, R39.1
- new net: R36.2, R39.2, R40.1
- new net: J5.3, R51.2, R55.1
- new net: R52.2, R55.2, R56.1
- new net: R37.2, R40.2, R41.1
- new net: R53.2, R56.2, R57.1
- new net: R38.2, R41.2, R42.1
- new net: J5.13, R59.1
- new net: R45.2, R48.2, R49.1
- new net: R44.2, R47.2, R48.1
- new net: J5.14, R60.1
- new net: J5.2, R43.2, R47.1
- new net: R54.2, R57.2, R58.1
- no-connect marks 3 -> 7
Other:
- note added: "Blue"
- note added: "Green"
- note added: "HSYNC"
- note added: "No shielding?"
- note added: "Red"
- note added: "See: https://digilent.com/reference/_media/reference/pmod/pmodvga/pmodvga_sch.pdf"
- note added: "TODO: Check footprint of these against datasheet, there is spooky buisness here"
- note added: "VSYNC"
- moved on the sheet: C39, C83, C84, C85, R16, R17, R18, R19, R20, R21, R24, R28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

Commit message: Renumber parts
Parts:
- renumbered C39 to C75, C83 to C76, C84 to C77, C85 to C78, J5 to J8, R16 to R28, R17 to R29, R18 to R30, R19 to R31, R20 to R32, R21 to R33, R24 to R34, R28 to R35, R29 to R36, R30 to R37, R31 to R38, R32 to R39, R33 to R40, R34 to R41, R35 to R42, R36 to R43, R37 to R44, R38 to R45, R39 to R46, R40 to R47, R41 to R48, R42 to R49, R43 to R50, R44 to R51, R45 to R52, R46 to R53, R47 to R54, R48 to R55, R49 to R56, R50 to R57, R51 to R58, R52 to R59, R53 to R60, R54 to R61, R55 to R62, R56 to R63, R57 to R64, R58 to R65, R59 to R66, R60 to R67, U7 to U6, U8 to U7

Commit message: footprints
Parts:
- removed J8: 1-1734530-3, MicroHard:CONN_1-1734530-1_TYCO, symbol VGA PORT:1-1734530-3
- added J?: L77HDE15SD1CH4FVGA, L77HDE15SD1CH4FVGA:AMPHENOL_L77HDE15SD1CH4FVGA, symbol L77HDE15SD1CH4FVGA:L77HDE15SD1CH4FVGA
- C75, C76, C77, C78: footprint (none) -> Capacitor_SMD:C_1206_3216Metric_Pad1.33x1.80mm_HandSolder
- R28, R29, R30, R31, R32, R33, R34, R35, R36, R37, R38, R39, R40, R41, R42, R43, R44, R45, R46, R47, R48, R49, R50, R51, R52, R53, R54, R55, R56, R57, R58, R59, R60, R61, R62, R63, R64, R65, R66, R67: footprint (none) -> Resistor_SMD:R_1206_3216Metric_Pad1.30x1.75mm_HandSolder
Connections:
- net GND: now also J?.10, J?.5, J?.6, J?.7, J?.8
- net at R42.2, R46.1: now also J?.1
- net at R58.2, R62.1: now also J?.3
- net at R50.2, R54.1: now also J?.2
- no-connect marks 7 -> 4
Other:
- note removed: "No shielding?"
- moved on the sheet: R66, R67

Commit message: added VGA footprint
Parts:
- added C81: 4p, Capacitor_SMD:C_1206_3216Metric_Pad1.33x1.80mm_HandSolder, symbol Device:C
- added R73: 1MEG, Resistor_SMD:R_1206_3216Metric_Pad1.30x1.75mm_HandSolder, symbol Device:R
- J8: renamed from J?; footprint L77HDE15SD1CH4FVGA:AMPHENOL_L77HDE15SD1CH4FVGA -> MicroHard:AMPHENOL_L77HDE15SD1CH4FVGA
Connections:
- net GND: now also C81.2, R73.2
- net at R66.1: now also J8.13
- net at R67.1: now also J8.14
- net at J8.SH1 (SHIELD): now also J8.SH2 (SHIELD__1), C81.1, R73.1
- no-connect marks 4 -> 7
Other:
- note added: "VGA_SHIELD"

Commit message: Initial layout
Parts:
- renumbered C77 to C76, C76 to C77, C81 to C79, R32 to R29, R36 to R30, R39 to R31, R42 to R32, R46 to R33, R43 to R34, R50 to R35, R29 to R36, R33 to R37, R37 to R38, R40 to R39, R47 to R40, R54 to R41, R44 to R42, R51 to R43, R58 to R44, R48 to R45, R55 to R46, R62 to R47, R45 to R48, R52 to R49, R59 to R50, R49 to R51, R56 to R52, R63 to R53, R53 to R54, R60 to R55, R57 to R56, R64 to R57, R61 to R58, R73 to R59, R65 to R60, R30 to R61, R34 to R62, R38 to R63, R41 to R64, R66 to R65, R67 to R66, R31 to R67, R35 to R68

Commit message: finished memory
Parts:
- removed R28, R29, R30, R31, R36, R37, R38, R39, R61, R62, R63, R64, R67, R68: 100k, Resistor_SMD:R_1206_3216Metric_Pad1.30x1.75mm_HandSolder, symbol Device:R

Commit message: Small fixes
Parts:
- C79: footprint Capacitor_SMD:C_1206_3216Metric_Pad1.33x1.80mm_HandSolder -> Capacitor_SMD:C_0805_2012Metric_Pad1.18x1.45mm_HandSolder
Changed lines of the file:
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@@
 			)
 		)
-		(property "Footprint" "Capacitor_SMD:C_1206_3216Metric_Pad1.33x1.80mm_HandSolder"
+		(property "Footprint" "Capacitor_SMD:C_0805_2012Metric_Pad1.18x1.45mm_HandSolder"
 			(at 266.3952 113.03 0)
 			(effects

Commit message: Fix schematics for delivery
Parts:
- C79: value 4p -> 1n
Other:
- company: (none) -> MicroHard
- title: (none) -> VGA
