File: MicroHardController/MicroHardController.kicad_pcb (KiCad board)
At the start: 2 copper layers, 4 parts, among them J1 Conn_01x07_Pin, SW1 SW_Push_LED, U1 THB001P

Commit message: feat: added EFM32GG842... schematic symbol
Routing:
- net Xout: track 124.8 -> 123.2 mm
Other:
- board outline added: 90.5 x 143.5 mm
Changed lines of the file:
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@@
 		)
 		(fp_text user "${REFERENCE}"
-			(at 0 7.62 360)
+			(at 0 7.62 0)
 			(layer "F.Fab")
 			(effects
@@
 		(tags "Through hole pin header THT 1x04 2.54mm single row")
 		(property "Reference" "SW1"
-			(at 0 -2.33 360)
+			(at 0 -2.33 0)
 			(layer "F.SilkS")
 			(effects
@@
 		)
 		(property "Value" "SW_Push_LED"
-			(at 0 9.95 360)
+			(at 0 9.95 0)
 			(layer "F.Fab")
 			(effects
@@
 		)
 	)
+	(gr_rect
+		(start 17 21)
+		(end 107.5 164.5)
+		(stroke
+			(width 0.05)
+			(type default)
+		)
+		(fill none)
+		(layer "Edge.Cuts")
+	)
 	(segment
 		(start 90.7 70)
@@
 	)
 	(segment
-		(start 99.4675 144.425)
-		(end 98.3425 145.55)
-		(width 0.2)
-		(layer "F.Cu")
-		(net 4)
-	)
-	(segment

Commit message: feat: controller fixed
Parts:
- added R1: 100K, Resistor_SMD:R_1206_3216Metric_Pad1.30x1.75mm_HandSolder, F.Cu at (101.0, 155.0)
- added R2: 100K, Resistor_SMD:R_1206_3216Metric_Pad1.30x1.75mm_HandSolder, F.Cu at (99.4, 74.0)
Connections:
- net Fbtn renamed Button1
- J1 pad 7: unconnected-(J1-Pin_7-Pad7) -> Button2
- U1 pad A: unconnected-(U1-a-PadA) -> +3.3VA
- U1 pad D: unconnected-(U1-d-PadD) -> Button2
Routing:
- net Button2: track 0.00 -> 139.9 mm
- net GND: track 193.2 -> 211.4 mm
- net +3.3VA: track 207.9 -> 213.3 mm
- net Button1: track 65.1 -> 70.1 mm
